File: 75-pixels.kicad_pcb (KiCad board)
At the start: 2 copper layers, 284.9 x 95.5 mm, 167 parts, among them J1 USB_B_Mini, J2 USB_B_Mini, J3 Conn_01x04, J4 USB_B_Mini, J5 Conn_01x04, SW1 SW_Push, U1 ProMicro, U2 ProMicro

Commit message: Update gerbers
Parts:
- removed the Poker_oval_hole at (299.7, 73.5)
- removed the Poker_oval_hole at (17.2, 73.7)
Routing:
- net col0: track 279.6 -> 285.0 mm
Other:
- outline, holes or cut-outs redrawn

Commit message: Move diodes
Parts:
- moved D4_8 20.6 mm to (207.7, 95.2)
- moved D4_6 20.4 mm to (169.2, 104.3), turned to 270 degrees
- moved D4_5 19.3 mm to (111.9, 105.8), turned to 270 degrees
- moved D4_9 18.8 mm to (225.2, 95.2)
Routing:
- net GND: track 61.7 -> 34.5 mm, vias 12 -> 14
- net Net-(D4_6-Pad2): track 6.46 -> 32.6 mm
- net Net-(D4_8-Pad2): track 4.52 -> 26.9 mm
- net row9: track 414.2 -> 393.8 mm, vias 7 -> 5
- net Net-(D4_9-Pad2): track 25.8 -> 46.1 mm
- net Net-(D4_5-Pad2): track 8.31 -> 19.2 mm
- net col5: track 310.0 -> 316.5 mm
- net row8: track 467.3 -> 467.1 mm, vias 4 -> 6
